Commit message: Update planner behavior, mapping config, and robot visuals

File: description/robot_core_lr.xacro (robot description, xacro)
@@ -8,4 +8,7 @@
 		<color rgba="0 0 0 1"/>
 	</material>
+	<material name="yellow">
+		<color rgba="1 1 0 1"/>
+	</material>
 	<!-- BASE LINK -->
 	<link name="base_link">
@@ -36,4 +39,13 @@
 	</joint>
 	<link name="chassis_link">
+		<visual>
+			<!-- Scale/offset STL to match LR collision body (~0.8 x 0.4 x 0.05 at z=0.1) -->
+			<origin xyz="0.5248 0.1928 0.1595" rpy="0 0 0"/>
+			<geometry>
+				<mesh filename="package://four_wheeled_robot/meshes/chassis_link.STL" scale="6.154 4.0 12.5"/>
+			</geometry>
+			<material name="white"/>
+		</visual>
+		<!-- Primitive fallback so the body is still visible if mesh rendering fails -->
 		<visual>
 			<origin xyz="0 0 0.1"/>
@@ -126,4 +138,19 @@
 	<link name="wheel1_link">
 		<visual>
+			<origin xyz="0 0 0.0167" rpy="0 0 0"/>
+			<geometry>
+				<mesh filename="package://four_wheeled_robot/meshes/wheel1_Link.STL" scale="2.56 2.56 3.333"/>
+			</geometry>
+			<material name="yellow"/>
+		</visual>
+		<visual>
+			<origin xyz="0 0 -0.005" rpy="0 0 0"/>
+			<geometry>
+				<mesh filename="package://four_wheeled_robot/meshes/tire1_Link.STL" scale="2.04 2.04 3.333"/>
+			</geometry>
+			<material name="black"/>
+		</visual>
+		<!-- Primitive fallback so wheel remains visible if mesh loading fails -->
+		<visual>
 			<geometry>
 				<cylinder radius="0.1" length="0.1"/>
@@ -154,4 +181,19 @@
 	<link name="wheel2_link">
 		<visual>
+			<origin xyz="0 0 0.0167" rpy="0 0 0"/>
+			<geometry>
+				<mesh filename="package://four_wheeled_robot/meshes/wheel2_Link.STL" scale="2.56 2.56 3.333"/>
+			</geometry>
+			<material name="yellow"/>
+		</visual>
+		<visual>
+			<origin xyz="0 0 -0.005" rpy="0 0 0"/>
+			<geometry>
+				<mesh filename="package://four_wheeled_robot/meshes/tire2_Link.STL" scale="2.04 2.04 3.333"/>
+			</geometry>
+			<material name="black"/>
+		</visual>
+		<!-- Primitive fallback so wheel remains visible if mesh loading fails -->
+		<visual>
 			<geometry>
 				<cylinder radius="0.1" length="0.1"/>
@@ -182,4 +224,19 @@
 	<link name="wheel3_link">
 		<visual>
+			<origin xyz="0 0 0.0167" rpy="0 0 0"/>
+			<geometry>
+				<mesh filename="package://four_wheeled_robot/meshes/wheel3_Link.STL" scale="2.56 2.56 3.333"/>
+			</geometry>
+			<material name="yellow"/>
+		</visual>
+		<visual>
+			<origin xyz="0 0 -0.005" rpy="0 0 0"/>
+			<geometry>
+				<mesh filename="package://four_wheeled_robot/meshes/tire3_Link.STL" scale="2.04 2.04 3.333"/>
+			</geometry>
+			<material name="black"/>
+		</visual>
+		<!-- Primitive fallback so wheel remains visible if mesh loading fails -->
+		<visual>
 			<geometry>
 				<cylinder radius="0.1" length="0.1"/>
@@ -210,4 +267,19 @@
 	<link name="wheel4_link">
 		<visual>
+			<origin xyz="0 0 0.0167" rpy="0 0 0"/>
+			<geometry>
+				<mesh filename="package://four_wheeled_robot/meshes/wheel4_Link.STL" scale="2.56 2.56 3.333"/>
+			</geometry>
+			<material name="yellow"/>
+		</visual>
+		<visual>
+			<origin xyz="0 0 0.045" rpy="0 0 0"/>
+			<geometry>
+				<mesh filename="package://four_wheeled_robot/meshes/tire4_Link.STL" scale="2.04 2.04 3.333"/>
+			</geometry>
+			<material name="black"/>
+		</visual>
+		<!-- Primitive fallback so wheel remains visible if mesh loading fails -->
+		<visual>
 			<geometry>
 				<cylinder radius="0.1" length="0.1"/>

Commit message: backup: snapshot 20260410-095914

File: description/robot_core_lr.xacro (robot description, xacro)
@@ -11,4 +11,6 @@
 		<color rgba="1 1 0 1"/>
 	</material>
+	<!-- DAE meshes keep the original visual look -->
+	<xacro:property name="elm_scale" value="1.0"/>
 	<!-- BASE LINK -->
 	<link name="base_link">
@@ -38,34 +40,43 @@
 		<origin xyz="0 0 0"/>
 	</joint>
-	<link name="chassis_link">
-		<visual>
-			<!-- Scale/offset STL to match LR collision body (~0.8 x 0.4 x 0.05 at z=0.1) -->
-			<origin xyz="0.5248 0.1928 0.1595" rpy="0 0 0"/>
-			<geometry>
-				<mesh filename="package://four_wheeled_robot/meshes/chassis_link.STL" scale="6.154 4.0 12.5"/>
+		<link name="chassis_link">
+		<visual>
+			<origin xyz="0 0 0" rpy="0 0 0"/>
+			<geometry>
+					<mesh filename="package://four_wheeled_robot/meshes/BaseMetal.dae" scale="${elm_scale} ${elm_scale} ${elm_scale}"/>
 			</geometry>
 			<material name="white"/>
 		</visual>
-		<!-- Primitive fallback so the body is still visible if mesh rendering fails -->
-		<visual>
-			<origin xyz="0 0 0.1"/>
-			<geometry>
-				<box size="0.8 0.4 0.05"/>
-			</geometry>
-			<material name="white"/>
-		</visual>
-		<collision>
-			<origin xyz="0 0 0.1"/>
-			<geometry>
-				<box size="0.8 0.4 0.05"/>
-			</geometry>
-		</collision>
-		<xacro:inertial_box mass="0.5" x="0.8" y="0.4" z="0.05">
-        	<origin xyz="0 0 0.1" rpy="0 0 0"/>
+		<visual>
+			<origin xyz="0 0 0" rpy="0 0 0"/>
+			<geometry>
+					<mesh filename="package://four_wheeled_robot/meshes/BaseRubber.dae" scale="${elm_scale} ${elm_scale} ${elm_scale}"/>
+			</geometry>
+			<material name="black"/>
+		</visual>
+		<visual>
+			<origin xyz="0 0 0" rpy="0 0 0"/>
+			<geometry>
+					<mesh filename="package://four_wheeled_robot/meshes/BasePlastic.dae" scale="${elm_scale} ${elm_scale} ${elm_scale}"/>
+			</geometry>
+			<material name="yellow"/>
+		</visual>
+			<visual>
+				<origin xyz="0 0 0" rpy="0 0 0"/>
+				<geometry>
+						<mesh filename="package://four_wheeled_robot/meshes/BaseClear.dae" scale="${elm_scale} ${elm_scale} ${elm_scale}"/>
+				</geometry>
+				<material name="white"/>
+			</visual>
+		<collision>
+			<origin xyz="0 0 0.0875"/>
+			<geometry>
+				<box size="0.8 0.389 0.171"/>
+			</geometry>
+		</collision>
+		<xacro:inertial_box mass="0.5" x="0.8" y="0.389" z="0.171">
+        	<origin xyz="0 0 0.0875" rpy="0 0 0"/>
         </xacro:inertial_box>
 	</link>
-	<gazebo reference="chassis_link">
-		<material>Gazebo/White</material>
-	</gazebo>
 	<!-- LIDAR -->
 	<joint name="lidar_joint" type="fixed">
@@ -92,9 +103,9 @@
         </xacro:inertial_cylinder>
 	</link>
-	<gazebo reference="lidar_link">
-		<sensor name="lidar_sensor" type="ray">
-			<always_on>true</always_on>
-			<visualize>true</visualize>
-			<update_rate>8</update_rate>
+		<gazebo reference="lidar_link">
+			<sensor name="lidar_sensor" type="ray">
+				<always_on>true</always_on>
+					<visualize>true</visualize>
+				<update_rate>8</update_rate>
 			<pose>0 0 0 0 0 0</pose>
 			<ray>
@@ -136,38 +147,28 @@
 	    <dynamics damping="1.0" friction="1.0" />
 	</joint>
-	<link name="wheel1_link">
-		<visual>
-			<origin xyz="0 0 0.0167" rpy="0 0 0"/>
-			<geometry>
-				<mesh filename="package://four_wheeled_robot/meshes/wheel1_Link.STL" scale="2.56 2.56 3.333"/>
-			</geometry>
-			<material name="yellow"/>
-		</visual>
-		<visual>
-			<origin xyz="0 0 -0.005" rpy="0 0 0"/>
-			<geometry>
-				<mesh filename="package://four_wheeled_robot/meshes/tire1_Link.STL" scale="2.04 2.04 3.333"/>
-			</geometry>
-			<material name="black"/>
-		</visual>
-		<!-- Primitive fallback so wheel remains visible if mesh loading fails -->
-		<visual>
-			<geometry>
-				<cylinder radius="0.1" length="0.1"/>
-			</geometry>
-			<material name="black"/>
-		</visual>
-		<collision>
-			<geometry>
-				<cylinder radius="0.1" length="0.1"/>
-			</geometry>
-		</collision>
-		<xacro:inertial_cylinder mass="0.1" length="0.1" radius="0.1">
-        	<origin xyz="0 0 0" rpy="0 0 0"/>
-        </xacro:inertial_cylinder>
-	</link>
-	<gazebo reference="wheel1_link">
-		<material>Gazebo/Black</material>
-	</gazebo>
+		<link name="wheel1_link">
+		<visual>
+			<origin xyz="0 0 0" rpy="0 0 ${pi}"/>
+			<geometry>
+					<mesh filename="package://four_wheeled_robot/meshes/HubMotor.dae" scale="${elm_scale} ${elm_scale} ${elm_scale}"/>
+			</geometry>
+			<material name="yellow"/>
+		</visual>
+			<visual>
+				<origin xyz="0 0 0" rpy="0 0 ${pi}"/>
+				<geometry>
+						<mesh filename="package://four_wheeled_robot/meshes/RubberWheel.dae" scale="${elm_scale} ${elm_scale} ${elm_scale}"/>
+				</geometry>
+				<material name="black"/>
+			</visual>
+		<collision>
+			<geometry>
+				<cylinder radius="0.1" length="0.1"/>
+			</geometry>
+		</collision>
+		<xacro:inertial_cylinder mass="0.1" length="0.1" radius="0.1">
+        	<origin xyz="0 0 0" rpy="0 0 0"/>
+        </xacro:inertial_cylinder>
+	</link>
 	<!-- WHEEL2 -->
 	<joint name="wheel2_joint" type="continuous">
@@ -179,38 +180,28 @@
 	    <dynamics damping="1.0" friction="1.0" />
 	</joint>
-	<link name="wheel2_link">
-		<visual>
-			<origin xyz="0 0 0.0167" rpy="0 0 0"/>
-			<geometry>
-				<mesh filename="package://four_wheeled_robot/meshes/wheel2_Link.STL" scale="2.56 2.56 3.333"/>
-			</geometry>
-			<material name="yellow"/>
-		</visual>
-		<visual>
-			<origin xyz="0 0 -0.005" rpy="0 0 0"/>
-			<geometry>
-				<mesh filename="package://four_wheeled_robot/meshes/tire2_Link.STL" scale="2.04 2.04 3.333"/>
-			</geometry>
-			<material name="black"/>
-		</visual>
-		<!-- Primitive fallback so wheel remains visible if mesh loading fails -->
-		<visual>
-			<geometry>
-				<cylinder radius="0.1" length="0.1"/>
-			</geometry>
-			<material name="black"/>
-		</visual>
-		<collision>
-			<geometry>
-				<cylinder radius="0.1" length="0.1"/>
-			</geometry>
-		</collision>
-		<xacro:inertial_cylinder mass="0.1" length="0.1" radius="0.1">
-        	<origin xyz="0 0 0" rpy="0 0 0"/>
-        </xacro:inertial_cylinder>
-	</link>
-	<gazebo reference="wheel2_link">
-		<material>Gazebo/Black</material>
-	</gazebo>
+		<link name="wheel2_link">
+		<visual>
+			<origin xyz="0 0 0" rpy="0 0 0"/>
+			<geometry>
+					<mesh filename="package://four_wheeled_robot/meshes/HubMotor.dae" scale="${elm_scale} ${elm_scale} ${elm_scale}"/>
+			</geometry>
+			<material name="yellow"/>
+		</visual>
+			<visual>
+				<origin xyz="0 0 0" rpy="0 0 0"/>
+				<geometry>
+						<mesh filename="package://four_wheeled_robot/meshes/RubberWheel.dae" scale="${elm_scale} ${elm_scale} ${elm_scale}"/>
+				</geometry>
+				<material name="black"/>
+			</visual>
+		<collision>
+			<geometry>
+				<cylinder radius="0.1" length="0.1"/>
+			</geometry>
+		</collision>
+		<xacro:inertial_cylinder mass="0.1" length="0.1" radius="0.1">
+        	<origin xyz="0 0 0" rpy="0 0 0"/>
+        </xacro:inertial_cylinder>
+	</link>
 	<!-- WHEEL3 -->
 	<joint name="wheel3_joint" type="continuous">
@@ -222,38 +213,28 @@
 	    <dynamics damping="1.0" friction="1.0" />
 	</joint>
-	<link name="wheel3_link">
-		<visual>
-			<origin xyz="0 0 0.0167" rpy="0 0 0"/>
-			<geometry>
-				<mesh filename="package://four_wheeled_robot/meshes/wheel3_Link.STL" scale="2.56 2.56 3.333"/>
-			</geometry>
-			<material name="yellow"/>
-		</visual>
-		<visual>
-			<origin xyz="0 0 -0.005" rpy="0 0 0"/>
-			<geometry>
-				<mesh filename="package://four_wheeled_robot/meshes/tire3_Link.STL" scale="2.04 2.04 3.333"/>
-			</geometry>
-			<material name="black"/>
-		</visual>
-		<!-- Primitive fallback so wheel remains visible if mesh loading fails -->
-		<visual>
-			<geometry>
-				<cylinder radius="0.1" length="0.1"/>
-			</geometry>
-			<material name="black"/>
-		</visual>
-		<collision>
-			<geometry>
-				<cylinder radius="0.1" length="0.1"/>
-			</geometry>
-		</collision>
-		<xacro:inertial_cylinder mass="0.1" length="0.1" radius="0.1">
-        	<origin xyz="0 0 0" rpy="0 0 0"/>
-        </xacro:inertial_cylinder>
-	</link>
-	<gazebo reference="wheel3_link">
-		<material>Gazebo/Black</material>
-	</gazebo>
+		<link name="wheel3_link">
+		<visual>
+			<origin xyz="0 0 0" rpy="0 0 ${pi}"/>
+			<geometry>
+					<mesh filename="package://four_wheeled_robot/meshes/HubMotor.dae" scale="${elm_scale} ${elm_scale} ${elm_scale}"/>
+			</geometry>
+			<material name="yellow"/>
+		</visual>
+			<visual>
+				<origin xyz="0 0 0" rpy="0 0 ${pi}"/>
+				<geometry>
+						<mesh filename="package://four_wheeled_robot/meshes/RubberWheel.dae" scale="${elm_scale} ${elm_scale} ${elm_scale}"/>
+				</geometry>
+				<material name="black"/>
+			</visual>
+		<collision>
+			<geometry>
+				<cylinder radius="0.1" length="0.1"/>
+			</geometry>
+		</collision>
+		<xacro:inertial_cylinder mass="0.1" length="0.1" radius="0.1">
+        	<origin xyz="0 0 0" rpy="0 0 0"/>
+        </xacro:inertial_cylinder>
+	</link>
 	<!-- WHEEL4 -->
 	<joint name="wheel4_joint" type="continuous">
@@ -265,37 +246,27 @@
 	    <dynamics damping="1.0" friction="1.0" />
 	</joint>
-	<link name="wheel4_link">
-		<visual>
-			<origin xyz="0 0 0.0167" rpy="0 0 0"/>
-			<geometry>
-				<mesh filename="package://four_wheeled_robot/meshes/wheel4_Link.STL" scale="2.56 2.56 3.333"/>
-			</geometry>
-			<material name="yellow"/>
-		</visual>
-		<visual>
-			<origin xyz="0 0 0.045" rpy="0 0 0"/>
-			<geometry>
-				<mesh filename="package://four_wheeled_robot/meshes/tire4_Link.STL" scale="2.04 2.04 3.333"/>
-			</geometry>
-			<material name="black"/>
-		</visual>
-		<!-- Primitive fallback so wheel remains visible if mesh loading fails -->
-		<visual>
-			<geometry>
-				<cylinder radius="0.1" length="0.1"/>
-			</geometry>
-			<material name="black"/>
-		</visual>
-		<collision>
-			<geometry>
-				<cylinder radius="0.1" length="0.1"/>
-			</geometry>
-		</collision>
-		<xacro:inertial_cylinder mass="0.1" length="0.1" radius="0.1">
-        	<origin xyz="0 0 0" rpy="0 0 0"/>
-        </xacro:inertial_cylinder>
-	</link>
-	<gazebo reference="wheel4_link">
-		<material>Gazebo/Black</material>
-	</gazebo>
-</robot>
+			<link name="wheel4_link">
+		<visual>
+			<origin xyz="0 0 0" rpy="0 0 0"/>
+			<geometry>
+					<mesh filename="package://four_wheeled_robot/meshes/HubMotor.dae" scale="${elm_scale} ${elm_scale} ${elm_scale}"/>
+			</geometry>
+			<material name="yellow"/>
+		</visual>
+			<visual>
+				<origin xyz="0 0 0" rpy="0 0 0"/>
+				<geometry>
+						<mesh filename="package://four_wheeled_robot/meshes/RubberWheel.dae" scale="${elm_scale} ${elm_scale} ${elm_scale}"/>
+				</geometry>
+				<material name="black"/>
+			</visual>
+		<collision>
+			<geometry>
+				<cylinder radius="0.1" length="0.1"/>
+			</geometry>
+		</collision>
+		<xacro:inertial_cylinder mass="0.1" length="0.1" radius="0.1">
+        	<origin xyz="0 0 0" rpy="0 0 0"/>
+	        </xacro:inertial_cylinder>
+		</link>
+	</robot>
