Commit message: release: v2.0

File: description/gazebo_control.xacro (robot description, xacro)
@@ -32,5 +32,5 @@
         <plugin name="four_wheel_joint_state" filename="libgazebo_ros_joint_state_publisher.so">
             <ros>
-                <remapping>~/out:=joint_states</remapping>
+                <remapping>~/out:=/joint_states</remapping>
             </ros>
             <update_rate>50</update_rate>

File: description/robot_core_lr.xacro (robot description, xacro)
@@ -2,12 +2,24 @@
 <robot xmlns:xacro="http://www.ros.org/wiki/xacro">
 	<xacro:include filename="inertial_macros.xacro"/>
-	<material name="white">
-		<color rgba="1 1 1 1"/>
-	</material>
-	<material name="black">
-		<color rgba="0 0 0 1"/>
-	</material>
-	<material name="yellow">
-		<color rgba="1 1 0 1"/>
+	<material name="chassis_metal">
+		<color rgba="0.18 0.22 0.27 1"/>
+	</material>
+	<material name="chassis_rubber">
+		<color rgba="0.03 0.03 0.04 1"/>
+	</material>
+	<material name="chassis_panel">
+		<color rgba="0.98 0.45 0.08 1"/>
+	</material>
+	<material name="chassis_clear">
+		<color rgba="0.55 0.75 0.95 0.45"/>
+	</material>
+	<material name="wheel_hub">
+		<color rgba="0.95 0.70 0.15 1"/>
+	</material>
+	<material name="wheel_tire">
+		<color rgba="0.02 0.02 0.02 1"/>
+	</material>
+	<material name="lidar_accent">
+		<color rgba="0.10 0.85 0.75 1"/>
 	</material>
 	<!-- DAE meshes keep the original visual look -->
@@ -46,5 +58,5 @@
 					<mesh filename="package://four_wheeled_robot/meshes/BaseMetal.dae" scale="${elm_scale} ${elm_scale} ${elm_scale}"/>
 			</geometry>
-			<material name="white"/>
+			<material name="chassis_metal"/>
 		</visual>
 		<visual>
@@ -53,5 +65,5 @@
 					<mesh filename="package://four_wheeled_robot/meshes/BaseRubber.dae" scale="${elm_scale} ${elm_scale} ${elm_scale}"/>
 			</geometry>
-			<material name="black"/>
+			<material name="chassis_rubber"/>
 		</visual>
 		<visual>
@@ -60,5 +72,5 @@
 					<mesh filename="package://four_wheeled_robot/meshes/BasePlastic.dae" scale="${elm_scale} ${elm_scale} ${elm_scale}"/>
 			</geometry>
-			<material name="yellow"/>
+			<material name="chassis_panel"/>
 		</visual>
 			<visual>
@@ -67,5 +79,5 @@
 						<mesh filename="package://four_wheeled_robot/meshes/BaseClear.dae" scale="${elm_scale} ${elm_scale} ${elm_scale}"/>
 				</geometry>
-				<material name="white"/>
+				<material name="chassis_clear"/>
 			</visual>
 		<collision>
@@ -91,5 +103,5 @@
 				<cylinder radius="0.03" length="0.04"/>
 			</geometry>
-			<material name="black"/>
+			<material name="lidar_accent"/>
 		</visual>
 		<collision>
@@ -129,10 +141,10 @@
 				</noise>
 			</ray>
-			<plugin name="gazebo_ros_lidar" filename="libgazebo_ros_ray_sensor.so">
-				<ros>
-					<remapping>~/out:=scan</remapping>
-				</ros>
-				<output_type>sensor_msgs/LaserScan</output_type>
-				<frame_name>lidar_link</frame_name>
+				<plugin name="gazebo_ros_lidar" filename="libgazebo_ros_ray_sensor.so">
+					<ros>
+						<remapping>~/out:=/four_wheeled_robot/scan</remapping>
+					</ros>
+					<output_type>sensor_msgs/LaserScan</output_type>
+					<frame_name>lidar_link</frame_name>
 			</plugin>
 		</sensor>
@@ -142,6 +154,6 @@
 		<parent link="base_link"/>
 		<child link="wheel1_link"/>
-		<origin xyz="0.2 0.25 0" rpy="${-pi/2} 0 0"/>
-		<axis xyz="0 0 1"/>
+		<origin xyz="0.2 0.25 0" rpy="0 0 0"/>
+		<axis xyz="0 1 0"/>
 		<limit effort="80" velocity="20" />
 	    <dynamics damping="1.0" friction="1.0" />
@@ -153,5 +165,5 @@
 					<mesh filename="package://four_wheeled_robot/meshes/HubMotor.dae" scale="${elm_scale} ${elm_scale} ${elm_scale}"/>
 			</geometry>
-			<material name="yellow"/>
+			<material name="wheel_hub"/>
 		</visual>
 			<visual>
@@ -160,14 +172,15 @@
 						<mesh filename="package://four_wheeled_robot/meshes/RubberWheel.dae" scale="${elm_scale} ${elm_scale} ${elm_scale}"/>
 				</geometry>
-				<material name="black"/>
-			</visual>
-		<collision>
-			<geometry>
-				<cylinder radius="0.1" length="0.1"/>
-			</geometry>
-		</collision>
-		<xacro:inertial_cylinder mass="0.1" length="0.1" radius="0.1">
-        	<origin xyz="0 0 0" rpy="0 0 0"/>
-        </xacro:inertial_cylinder>
+				<material name="wheel_tire"/>
+			</visual>
+		<collision>
+			<origin xyz="0 0 0" rpy="${pi/2} 0 0"/>
+			<geometry>
+				<cylinder radius="0.1" length="0.1"/>
+			</geometry>
+		</collision>
+		<xacro:inertial_cylinder mass="0.1" length="0.1" radius="0.1">
+	        	<origin xyz="0 0 0" rpy="${pi/2} 0 0"/>
+	        </xacro:inertial_cylinder>
 	</link>
 	<!-- WHEEL2 -->
@@ -175,6 +188,6 @@
 		<parent link="base_link"/>
 		<child link="wheel2_link"/>
-		<origin xyz="0.2 -0.25 0" rpy="${pi/2} 0 0"/>
-		<axis xyz="0 0 -1"/>
+		<origin xyz="0.2 -0.25 0" rpy="0 0 0"/>
+		<axis xyz="0 1 0"/>
 		<limit effort="80" velocity="20" />
 	    <dynamics damping="1.0" friction="1.0" />
@@ -186,5 +199,5 @@
 					<mesh filename="package://four_wheeled_robot/meshes/HubMotor.dae" scale="${elm_scale} ${elm_scale} ${elm_scale}"/>
 			</geometry>
-			<material name="yellow"/>
+			<material name="wheel_hub"/>
 		</visual>
 			<visual>
@@ -193,14 +206,15 @@
 						<mesh filename="package://four_wheeled_robot/meshes/RubberWheel.dae" scale="${elm_scale} ${elm_scale} ${elm_scale}"/>
 				</geometry>
-				<material name="black"/>
-			</visual>
-		<collision>
-			<geometry>
-				<cylinder radius="0.1" length="0.1"/>
-			</geometry>
-		</collision>
-		<xacro:inertial_cylinder mass="0.1" length="0.1" radius="0.1">
-        	<origin xyz="0 0 0" rpy="0 0 0"/>
-        </xacro:inertial_cylinder>
+				<material name="wheel_tire"/>
+			</visual>
+		<collision>
+			<origin xyz="0 0 0" rpy="${pi/2} 0 0"/>
+			<geometry>
+				<cylinder radius="0.1" length="0.1"/>
+			</geometry>
+		</collision>
+		<xacro:inertial_cylinder mass="0.1" length="0.1" radius="0.1">
+	        	<origin xyz="0 0 0" rpy="${pi/2} 0 0"/>
+	        </xacro:inertial_cylinder>
 	</link>
 	<!-- WHEEL3 -->
@@ -208,6 +222,6 @@
 		<parent link="base_link"/>
 		<child link="wheel3_link"/>
-		<origin xyz="-0.2 0.25 0" rpy="${-pi/2} 0 0"/>
-		<axis xyz="0 0 1"/>
+		<origin xyz="-0.2 0.25 0" rpy="0 0 0"/>
+		<axis xyz="0 1 0"/>
 		<limit effort="80" velocity="20" />
 	    <dynamics damping="1.0" friction="1.0" />
@@ -219,5 +233,5 @@
 					<mesh filename="package://four_wheeled_robot/meshes/HubMotor.dae" scale="${elm_scale} ${elm_scale} ${elm_scale}"/>
 			</geometry>
-			<material name="yellow"/>
+			<material name="wheel_hub"/>
 		</visual>
 			<visual>
@@ -226,14 +240,15 @@
 						<mesh filename="package://four_wheeled_robot/meshes/RubberWheel.dae" scale="${elm_scale} ${elm_scale} ${elm_scale}"/>
 				</geometry>
-				<material name="black"/>
-			</visual>
-		<collision>
-			<geometry>
-				<cylinder radius="0.1" length="0.1"/>
-			</geometry>
-		</collision>
-		<xacro:inertial_cylinder mass="0.1" length="0.1" radius="0.1">
-        	<origin xyz="0 0 0" rpy="0 0 0"/>
-        </xacro:inertial_cylinder>
+				<material name="wheel_tire"/>
+			</visual>
+		<collision>
+			<origin xyz="0 0 0" rpy="${pi/2} 0 0"/>
+			<geometry>
+				<cylinder radius="0.1" length="0.1"/>
+			</geometry>
+		</collision>
+		<xacro:inertial_cylinder mass="0.1" length="0.1" radius="0.1">
+	        	<origin xyz="0 0 0" rpy="${pi/2} 0 0"/>
+	        </xacro:inertial_cylinder>
 	</link>
 	<!-- WHEEL4 -->
@@ -241,6 +256,6 @@
 		<parent link="base_link"/>
 		<child link="wheel4_link"/>
-		<origin xyz="-0.2 -0.25 0" rpy="${pi/2} 0 0"/>
-		<axis xyz="0 0 -1"/>
+		<origin xyz="-0.2 -0.25 0" rpy="0 0 0"/>
+		<axis xyz="0 1 0"/>
 		<limit effort="80" velocity="20" />
 	    <dynamics damping="1.0" friction="1.0" />
@@ -252,5 +267,5 @@
 					<mesh filename="package://four_wheeled_robot/meshes/HubMotor.dae" scale="${elm_scale} ${elm_scale} ${elm_scale}"/>
 			</geometry>
-			<material name="yellow"/>
+			<material name="wheel_hub"/>
 		</visual>
 			<visual>
@@ -259,13 +274,14 @@
 						<mesh filename="package://four_wheeled_robot/meshes/RubberWheel.dae" scale="${elm_scale} ${elm_scale} ${elm_scale}"/>
 				</geometry>
-				<material name="black"/>
-			</visual>
-		<collision>
-			<geometry>
-				<cylinder radius="0.1" length="0.1"/>
-			</geometry>
-		</collision>
-		<xacro:inertial_cylinder mass="0.1" length="0.1" radius="0.1">
-        	<origin xyz="0 0 0" rpy="0 0 0"/>
+				<material name="wheel_tire"/>
+			</visual>
+		<collision>
+			<origin xyz="0 0 0" rpy="${pi/2} 0 0"/>
+			<geometry>
+				<cylinder radius="0.1" length="0.1"/>
+			</geometry>
+		</collision>
+		<xacro:inertial_cylinder mass="0.1" length="0.1" radius="0.1">
+	        	<origin xyz="0 0 0" rpy="${pi/2} 0 0"/>
 	        </xacro:inertial_cylinder>
 		</link>
